File: M032FC1AE.kicad_pcb (KiCad board)
At the start: 2 copper layers, 27 parts, among them J1 Conn_01x10, J2 Conn_01x03, J3 Conn_01x04, J4 USB_C_Receptacle_USB2.0_16P, J5 Conn_01x03, J6 Conn_01x05, J7 Conn_02x08_Odd_Even, Q1 S8050, SW1 SW_Push, SW2 SW_Push, U1 AMS1117-1.8, U2 AMS1117-3.3, U3 USBLC6-2SC6

Commit message: fffff
Parts:
- added IC1: M032FC1AE, M032FC1AE:M032FC1AE, F.Cu at (69.9, 113.1)
- added R10: 330, Resistor_SMD:R_0603_1608Metric_Pad0.98x0.95mm_HandSolder, F.Cu at (69.9, 43.7)
- added R11: 330, Resistor_SMD:R_0603_1608Metric_Pad0.98x0.95mm_HandSolder, F.Cu at (69.9, 46.2)
- added R12: 330, Resistor_SMD:R_0603_1608Metric_Pad0.98x0.95mm_HandSolder, F.Cu at (69.9, 48.7)
- added R13: 330, Resistor_SMD:R_0603_1608Metric_Pad0.98x0.95mm_HandSolder, F.Cu at (69.9, 51.2)
- added R6: 330, Resistor_SMD:R_0603_1608Metric_Pad0.98x0.95mm_HandSolder, F.Cu at (69.9, 33.6)
- added R7: 330, Resistor_SMD:R_0603_1608Metric_Pad0.98x0.95mm_HandSolder, F.Cu at (69.9, 36.1)
- added R8: 330, Resistor_SMD:R_0603_1608Metric_Pad0.98x0.95mm_HandSolder, F.Cu at (69.9, 38.6)
- added R9: 330, Resistor_SMD:R_0603_1608Metric_Pad0.98x0.95mm_HandSolder, F.Cu at (69.9, 41.2)
Connections:
- J7 pad 1: unconnected-(J7-Pin_1-Pad1) -> spi_ss
- J7 pad 10: unconnected-(J7-Pin_10-Pad10) -> VCC
- J7 pad 11: unconnected-(J7-Pin_11-Pad11) -> Net-(J7-Pin_11)
- J7 pad 12: unconnected-(J7-Pin_12-Pad12) -> Net-(J7-Pin_12)
- J7 pad 13: unconnected-(J7-Pin_13-Pad13) -> Net-(J7-Pin_13)
- J7 pad 14: unconnected-(J7-Pin_14-Pad14) -> usci1_clk
- J7 pad 15: unconnected-(J7-Pin_15-Pad15) -> GND
- J7 pad 16: unconnected-(J7-Pin_16-Pad16) -> usci1_data
- J7 pad 2: unconnected-(J7-Pin_2-Pad2) -> VCC
- J7 pad 3: unconnected-(J7-Pin_3-Pad3) -> spi_miso
- J7 pad 4: unconnected-(J7-Pin_4-Pad4) -> Net-(J7-Pin_4)
- J7 pad 5: unconnected-(J7-Pin_5-Pad5) -> Net-(J7-Pin_5)
- J7 pad 6: unconnected-(J7-Pin_6-Pad6) -> spi_clk
- J7 pad 7: unconnected-(J7-Pin_7-Pad7) -> GND
- J7 pad 8: unconnected-(J7-Pin_8-Pad8) -> spi_mosi
- J7 pad 9: unconnected-(J7-Pin_9-Pad9) -> Net-(J7-Pin_9)
- R3 pad 1: VDD -> VCC

Commit message: ddddd
Parts:
- removed J3: Conn_01x04, Connector_PinHeader_2.54mm:PinHeader_1x04_P2.54mm_Horizontal
- J6: moved to B.Cu
- Q1: footprint Package_TO_SOT_THT:TO-92_Inline -> Package_TO_SOT_SMD:TSOT-23
- moved J1 116.0 mm to (174.2, 118.8), turned to -90 degrees
- moved J7 110.6 mm to (171.8, 98.2), turned to -90 degrees
- moved IC1 103.3 mm to (168.2, 81.4)
- moved J2 98.4 mm to (180.2, 113.7)
- moved J6 95.1 mm to (182.2, 78.4), turned to 180 degrees
- moved J4 86.3 mm to (160.2, 62.2), turned to 180 degrees
- moved C5 85.2 mm to (176.2, 79.7), turned to 90 degrees
- moved SW2 83.9 mm to (174.9, 70.0)
- moved SW1 83.7 mm to (174.9, 60.0)
- moved R1 82.1 mm to (178.0, 89.6), turned to -90 degrees
- moved C1 77.9 mm to (168.1, 65.4)
- moved R2 75.5 mm to (171.5, 89.7), turned to -90 degrees
- moved D1 72.5 mm to (176.6, 86.3), turned to 90 degrees
- moved Q1 72.3 mm to (174.8, 89.5)
- moved C2 72.2 mm to (163.4, 74.2), turned to 90 degrees
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Connections:
- C4 pad 1: Net-(J5-Pin_3) -> +3.3V
- J5 pad 3: Net-(J5-Pin_3) -> +3.3V
- U2 pad 2: Net-(J5-Pin_3) -> +3.3V

Commit message: ddddd
Parts:
- J6: moved to F.Cu
- moved R3 77.2 mm to (177.4, 83.3), turned to 90 degrees
- moved D1 27.2 mm to (149.6, 89.5)
- moved J6 11.6 mm to (180.2, 89.8)
- moved R2 7.57 mm to (175.6, 83.3)
- moved Q1 2.79 mm to (176.4, 87.3), turned to -90 degrees
- moved R1 1.86 mm to (176.4, 90.5), turned to 180 degrees
- moved C5 1.21 mm to (177.4, 79.8)

Commit message: ffffddd
Change-Id: I1eeee01593b08b9acbec1eab3a106692ce76c6c6
Parts:
- J7: value Conn_02x08_Odd_Even -> Conn_02x08_Counter_Clockwise
- moved R7 127.4 mm to (171.6, 112.7), turned to -90 degrees
- moved R6 114.0 mm to (169.1, 89.9), turned to -90 degrees
- moved R11 113.2 mm to (161.5, 112.7), turned to -90 degrees
- moved R12 109.7 mm to (158.9, 112.7), turned to 90 degrees
- moved R8 107.2 mm to (164.0, 89.9), turned to -90 degrees
- moved R13 106.2 mm to (156.4, 112.7), turned to 90 degrees
- moved R9 103.7 mm to (161.5, 89.9), turned to -90 degrees
- moved R10 100.3 mm to (158.9, 89.9), turned to -90 degrees
- moved R4 71.0 mm to (167.8, 60.2), turned to 90 degrees
- moved R5 57.8 mm to (152.6, 60.2), turned to 90 degrees
- moved J7 2.45 mm to (174.2, 97.5)
- moved C6 1.48 mm to (160.6, 81.1), turned to 180 degrees
- moved C7 1.12 mm to (160.6, 79.2), turned to 180 degrees
- moved J6 0.32 mm to (180.5, 89.8)
- moved J2 0.31 mm to (180.5, 113.7)
Connections:
- J1 pad 8: isci1_clk -> usci1_clk
- J7 pad 10: VCC -> usci1_clk
- J7 pad 12: Net-(J7-Pin_12) -> VCC
- J7 pad 13: Net-(J7-Pin_13) -> spi_mosi
- J7 pad 14: usci1_clk -> spi_clk
- J7 pad 15: GND -> Net-(J7-Pin_15)
- J7 pad 16: usci1_data -> VCC
- J7 pad 2: VCC -> spi_miso
- J7 pad 3: spi_miso -> Net-(J7-Pin_3)
- J7 pad 4: Net-(J7-Pin_4) -> GND
- J7 pad 6: spi_clk -> Net-(J7-Pin_6)
- J7 pad 7: GND -> Net-(J7-Pin_7)
- J7 pad 8: spi_mosi -> GND
- J7 pad 9: Net-(J7-Pin_9) -> usci1_data
- R10 pad 2: Net-(J7-Pin_13) -> Net-(J7-Pin_7)
- R11 pad 1: Net-(J7-Pin_12) -> Net-(J7-Pin_11)
- R6 pad 2: Net-(J7-Pin_5) -> Net-(J7-Pin_3)
- R7 pad 1: Net-(J7-Pin_4) -> Net-(J7-Pin_15)
- R8 pad 2: Net-(J7-Pin_9) -> Net-(J7-Pin_5)
- R9 pad 2: Net-(J7-Pin_11) -> Net-(J7-Pin_6)
Routing:
- net VCC: track 0.00 -> 146.4 mm, vias 0 -> 3
- net usci1_data: track 0.00 -> 61.4 mm, vias 0 -> 1
- net usci1_clk: track 0.00 -> 57.5 mm, vias 0 -> 1
- net VBUS: track 0.00 -> 52.1 mm, vias 0 -> 2
- net spi_clk: track 0.00 -> 50.0 mm
- net spi_miso: track 0.00 -> 47.4 mm, vias 0 -> 1
- net spi_mosi: track 0.00 -> 41.2 mm
- net spi_ss: track 0.00 -> 39.9 mm
- net uart_tx: track 0.00 -> 37.5 mm
- net rst: track 0.00 -> 36.7 mm
- net uart_rx: track 0.00 -> 35.0 mm
- net Net-(D1-K): track 0.00 -> 31.1 mm, vias 0 -> 1
- net +3.3V: track 0.00 -> 29.7 mm
- net ISP: track 0.00 -> 27.1 mm
- net GND: track 0.00 -> 26.3 mm, vias 0 -> 21
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- added copper zone on B.Cu, net GND
- added copper zone on F.Cu, net GND
Other:
- board outline added: 40.6 x 66 mm
- board text added: "GND"
- board text added: "I2C_CLK"
- board text added: "I2C_DAT"
- board text added: "RXD"
- board text added: "SPI_CLK"
- board text added: "SPI_MISO"
- board text added: "SPI_MOSI"
- board text added: "SPI_SS"
- board text added: "TXD"
- board text added: "VCC"

Commit message: dfdfdfdf
Change-Id: I4bedd6ca326a9b17d3d6f978c0846dd558e38f70
Parts:
- renumbered U1 to 1117-1V8, U2 to 1117-3V3, SW2 to ISP, SW1 to RST
Connections:
- J1 pad 4: spi_miso -> spi_mosi
- J1 pad 5: spi_mosi -> spi_miso
- J7 pad 13: spi_mosi -> spi_miso
- J7 pad 2: spi_miso -> spi_mosi
Routing:
- net spi_clk: track 50.0 -> 45.2 mm, vias 0 -> 1
- net spi_mosi: track 41.2 -> 45.9 mm, vias 0 -> 1
- net spi_miso: track 47.4 -> 42.8 mm
- net GND: vias 21 -> 25
Other:
- board text added: "1V8"
- board text added: "24xx"
- board text added: "25xx"
- board text added: "3V3"
- board text added: "A0"
- board text added: "A1"
- board text added: "A2"
- board text added: "CLK"
- board text added: "DAT"
- board text added: "DI"
- board text added: "DO"
- board text added: "HOLD"
- board text added: "I2C"
- board text added: "SPI"
- board text added: "SS"
- board text added: "WP"
