File: M032FC1AE.kicad_pcb (KiCad board)
At the start: 2 copper layers, 40.6 x 66 mm, 41 parts, among them IC1 M032FC1AE, J1 Conn_01x10, J2 Conn_01x03, J4 USB_C_Receptacle_USB2.0_16P, J5 Conn_01x03, J6 Conn_01x05, J7 Conn_02x08_Counter_Clockwise, Q2 SS8050, Q3 FDN340P, Q4 SS8550, SW1 SW_Push, SW2 SW_Push, U1 AMS1117-1.8, U2 AMS1117-3.3, U3 USBLC6-2SC6

Commit message: Release Gerver V0.1
Change-Id: If113fa1b5dadd0f7a6d01bb5205053d055243908
Parts:
- renumbered SW2 to ISP, D2 to ISP/PRG, U1 to LM1117_1V8, U2 to LM1117_3V3, SW1 to RST
Connections:
- net spi_clk renamed bus_spi_clk
- net spi_miso renamed bus_spi_miso
- net spi_mosi renamed bus_spi_mosi
- net spi_ss renamed bus_spi_ss
- net usci1_clk renamed bus_usci1_clk
- net usci1_data renamed bus_usci1_data
Routing:
- net bus_spi_ss: track 39.9 -> 56.7 mm
- net bus_spi_clk: track 45.2 -> 54.8 mm
- net bus_spi_mosi: track 48.4 -> 56.9 mm
- net bus_spi_miso: track 48.3 -> 54.0 mm
- net bus_usci1_clk: track 57.5 -> 62.8 mm
- net ice_clk: track 19.0 -> 20.0 mm
Other:
- board text added: "ICE_CLK"
- board text added: "ICE_DAT"
- board text added: "M032FC1AE Rom Programer V0.1"
- board text added: "RST"
