File: M032FC1AE.kicad_sch (KiCad schematic)
At the start: 21 parts, among them IC1 M032FC1AE, J1 Conn_01x10, J2 Conn_01x03, J3 Conn_01x04, Q1 S8050, SW1 SW_Push, SW2 SW_Slide_DPDT, U1 AMS1117-1.8, U2 AMS1117-3.3

Commit message: fff
Parts:
- removed SW2: SW_Slide_DPDT, Button_Switch_THT:SW_E-Switch_EG2219_DPDT_Angled, symbol Switch:SW_Slide_DPDT
- added C9: 1uf, Capacitor_SMD:C_0603_1608Metric_Pad1.08x0.95mm_HandSolder, symbol Device:C
- added J4: USB_C_Receptacle_USB2.0_16P, symbol Connector:USB_C_Receptacle_USB2.0_16P
- added J5: Conn_01x03, symbol Connector_Generic:Conn_01x03
Connections:
- net GND: now also C9.2, J4.A1 (GND), J4.A12 (GND), J4.B1 (GND), J4.B12 (GND), J4.S1 (SHIELD)
- net VBUS: now reaches C3.1, U2.3 (VI)
- net VBUS: now also C1.1, IC1.20 (USB_VBUS), U1.3 (VI), J4.A4 (VBUS), J4.A9 (VBUS), J4.B4 (VBUS), J4.B9 (VBUS)
- net at C4.1, U2.2 (VO): now also J5.3 (Pin_3)
- net VCC: now reaches IC1.10 (AVDD)
- net VCC: now also C7.1, IC1.3 (USB_VDD33_CAP), IC1.6 (VDD), C9.1, J5.2 (Pin_2)
- net spi_clk: now reaches IC1.7 (PB.14)
- net spi_miso: now reaches IC1.8 (PB.13)
- net spi_mosi: now reaches IC1.9 (PB.12)
- net at C2.1, U1.2 (VO): now also J5.1 (Pin_1)
Other:
- moved on the sheet: D1, IC1, Q1, R1, R2

Commit message: ddd
Change-Id: I6d4370392eb8b31b3cfbca76c540ab61eec68797
Parts:
- removed C8: 1uf, Capacitor_SMD:C_0603_1608Metric_Pad1.08x0.95mm_HandSolder, symbol Device:C
- added R4, R5: 5.1k, Resistor_SMD:R_0603_1608Metric_Pad0.98x0.95mm_HandSolder, symbol Device:R
- added U3: USBLC6-2SC6, Package_TO_SOT_SMD:SOT-23-6, symbol Power_Protection:USBLC6-2SC6
Connections:
- net GND: now also IC1.4 (VSS), J1.10 (Pin_10), J1.6 (Pin_6), J2.3 (Pin_3), R4.2, R5.2, U3.2 (GND)
- net VBUS: now also U3.5 (VBUS)
- net VCC: now also J1.1 (Pin_1), J1.7 (Pin_7)
- net ice_clk: now also IC1.19 (PF.1)
- net ice_dat: now also IC1.18 (PF.0)
- net isci1_clk: now also IC1.15 (PA.1), J1.8 (Pin_8)
- net rst: now also C5.1, IC1.17 (NRESET), R3.2, SW1.2
- net spi_clk: now also J1.3 (Pin_3)
- net spi_miso: now also J1.4 (Pin_4)
- net spi_mosi: now also J1.5 (Pin_5)
- net spi_ss: now also IC1.13 (PA.3), J1.2 (Pin_2)
- net uart_rx: now also IC1.12 (PF.2), J2.1 (Pin_1)
- net uart_tx: now also IC1.11 (PF.3), J2.2 (Pin_2)
- net usci1_data: now also IC1.14 (PA.2), J1.9 (Pin_9)
- net ISP: now reaches R2.1
- net ISP: now also IC1.16 (PA.0)
- net USB_D-: now reaches IC1.1 (USB_D-)
- net USB_D-: now also U3.6 (I/O1)
- net USB_D+: now reaches IC1.2 (USB_D+)
- net USB_D+: now also U3.4 (I/O2)
- net at J4.A5 (CC1): now also R4.1
- net at J4.A6 (D+): now also J4.B6 (D+), U3.3 (I/O2)
- net at J4.A7 (D-): now also J4.B7 (D-), U3.1 (I/O1)
- net at J4.B5 (CC2): now also R5.1
Other:
- moved on the sheet: C1, C2, C3, C4, C5, D1, J1, J2, J5, Q1, R1, R2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

Commit message: ffffff
Change-Id: Iabad5a04cb170e8d042da6a43dea56d0837ca319
Parts:
- added J6: Conn_01x05, Connector_PinSocket_2.54mm:PinSocket_1x05_P2.54mm_Horizontal, symbol Connector_Generic:Conn_01x05
- added J7: Conn_02x08_Odd_Even, Socket:DIP_Socket-16_W4.3_W5.08_W7.62_W10.16_W10.9_3M_216-3340-00-0602J, symbol Connector_Generic:Conn_02x08_Odd_Even
- added SW2: SW_Push, Button_Switch_THT:SW_PUSH_6mm, symbol Switch:SW_Push
- J4: footprint (none) -> Connector_USB:USB_C_Receptacle_GCT_USB4105-xx-A_16P_TopMnt_Horizontal
- J5: footprint (none) -> Connector_PinHeader_2.54mm:PinHeader_1x03_P2.54mm_Vertical
Connections:
- net GND: now also J6.5 (Pin_5), SW2.1
- net ISP: now also SW2.2
- net VCC: now also J6.1 (Pin_1); no longer C7.1, IC1.3 (USB_VDD33_CAP)
- net ice_clk: now also J6.3 (Pin_3)
- net ice_dat: now also J6.2 (Pin_2)
- net rst: now also J6.4 (Pin_4)
- new net: C7.1, IC1.3 (USB_VDD33_CAP)

Commit message: fffff
Parts:
- removed J3: Conn_01x04, Connector_PinHeader_2.54mm:PinHeader_1x04_P2.54mm_Horizontal, symbol Connector_Generic:Conn_01x04
- added R10, R11, R12, R13, R6, R7, R8, R9: 330, Resistor_SMD:R_0603_1608Metric_Pad0.98x0.95mm_HandSolder, symbol Device:R
- IC1: footprint SOP65P640X120-20N -> M032FC1AE:M032FC1AE
Connections:
- net VDD is gone; now on net VCC: R3.1
- net GND: now also J7.15 (Pin_15), J7.7 (Pin_7), R10.1, R11.2, R8.1, R9.1
- net VCC: now also J7.10 (Pin_10), J7.2 (Pin_2), R12.1, R13.1, R6.1, R7.2
- net isci1_clk: no longer IC1.15 (PA.1)
- net spi_clk: now also J7.6 (Pin_6)
- net spi_miso: now also J7.3 (Pin_3)
- net spi_mosi: now also J7.8 (Pin_8)
- net spi_ss: now also J7.1 (Pin_1)
- net usci1_data: now also J7.16 (Pin_16), R13.2
- net at J7.11 (Pin_11): now also R9.2
- net at J7.12 (Pin_12): now also R11.1
- net at J7.13 (Pin_13): now also R10.2
- net usci1_clk: now reaches J7.14 (Pin_14)
- net usci1_clk: now also IC1.15 (PA.1), R12.2
- net at J7.4 (Pin_4): now also R7.1
- net at J7.5 (Pin_5): now also R6.2
- net at J7.9 (Pin_9): now also R8.2
- no-connect marks 0 -> 2

Commit message: ddddd
Parts:
- Q1: footprint Package_TO_SOT_THT:TO-92_Inline -> Package_TO_SOT_SMD:TSOT-23
Connections:
- net +3.3V: now also C4.1, J5.3 (Pin_3), U2.2 (VO)
Changed lines of the file:
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@@
 	(wire
 		(pts
+			(xy 143.51 173.99) (xy 143.51 177.8)
+		)
+		(stroke
+			(width 0)
+			(type default)
+		)
+	)
+	(wire
+		(pts
 			(xy 26.67 97.79) (xy 26.67 102.87)
 		)
@@
 			"CgS0OnLR54qm9oKBNw2LcVrAWGiMVZ3nOelheFwZtw0LZ7D4chIUcEOVNdSHSXQqG2DT+Cs/9xPn"
 			"C/vPNOEA2wDRf7emMIQCjzCEAo8whALPoE1C7AmB7JcOKvwVQkHvjsJg3IL/B3tsWY+fUFgUAAAA"
-			"AElFTkSuQmCC"
+			"AElFTkSuQmCCAAAAAAAAAAAAAAAAAAAAAAAAAAAAAAAAAAAAAAAAAAAAAAAAAAAAAAAAAAAAAAAA"
+			"AAAAAAAAAAAAAAAAAAAAAAAAAAAAAAAAAAAAAAAAAAAAAAAAAAAAAAAAAAAAAAAAAAAAAAAAAAAA"
+			"AAAAAAAAAAAAAAAAAAAAAAAAAAAAAAAAAAAAAAAAAAAAAAAAAAAAAAAAAAAAAAAAAAAAAAAAAAAA"
+			"AAAAAAAAAAAAAAAAAAAAAAAAAAAAAAAAAAAAAAAAAAAAAAAAAAAAAAAAAAAAAAAAAAAAAAAAAAAA"
+			"AAAAAAAAAAAAAAAAAAAAAAAAAAAAAAAAAAAAAAAAAAAAAAAAAAAAAAAAAAAAAAAAAAAAAAAAAAAA"
+			"AAAAAAAAAAAAAAAAAAAAAAAAAAAAAAAAAAAAAAAAAAAAAAAAAAAAAAAAAAAAAAAAAAAAAAAAAAAA"
+			"AAAAAAAAAAAAAAAAAAAAAAAAAAAAAAAAAAAAAAAAAAAAAAAAAAAAAAAAAAAAAAAAAAAAAAAAAAAA"
+			"AAAAAAAAAAAAAAAAAAAAAAAAAAAAAAAAAAAAAAAAAAAAAAAAAAAAAAAAAAAAAAAAAAAAAAAAAAAA"
+			"AAAAAAAAAAAAAAAAAAAAAAAAAAAAAAAAAAAAAAAAAAAAAAAAAAAAAAAAAAAAAAAAAAAAAAAAAAAA"
+			"AAAAAAAAAAAAAAAAAAAAAAAAAAAAAAAAAAAAAAAAAAAAAAAAAAAAAAAAAAAAAAAAAAAAAAAAAAAA"
+			"AAAAAAAAAAAAAAAAAAAAAAAAAAAAAAAAAAAAAAAAAAAAAAAAAAAAAAAAAAAAAAAAAAAAAAAAAAAA"
+			"AAAAAAAAAAAAAAAAAAAAAAAAAAAAAAAAAAAAAAAAAAAAAAAAAAAAAAAAAAAAAAAAAAAAAAAAAAAA"
+			"AAAAAAAAAAAAAAAAAAAAAAAAAAAAAAAAAAAAAAAAAAAAAAAAAAAAAAAAAAAAAAAAAAAAAAAAAAAA"
+			"AAAAAAAAAAAAAAAAAAAAAAAAAAAAAAAAAAAAAAAAAAAAAAAAAAAAAAAAAAAAAAAAAAAAAAAAAAAA"
+			"AAAAAAAAAAAAAAAAAAAAAAAAAAAAAAAAAAAAAAAAAAAAAAAAAAAAAAAAAAAAAAAAAAAAAAAAAAAA"
+			"AAAAAAAAAAAAAAAAAAAAAAAAAAAAAAAAAAAAAAAAAAAAAAAAAAAAAAAAAAAAAAAAAAAAAAAAAAAA"
+			"AAAAAAAAAAAAAAAAAAAAAAAAAAAAAAAAAAAAAAAAAAAAAAAAAAAAAAAAAAAAAAAAAAAAAAAAAAAA"
+			"AAAAAAAAAAAAAAAAAAAAAAAAAAAAAAAAAAAAAAAAAAAAAAAAAAAAAAAAAAAAAAAAAAAAAAAAAAAA"
+			"AAAAAFCirQ=="
 		)
 	)
@@
 			"AAAAAAAAAAAAAAAAAAAAAAAAAAAAAAAAAAAAAAAAAAAAAAAAAAAAAAAAAAAAAAAAAAAAAAAAAAAA"
 			"AAAAAAAAAAAAAAAAAAAAAAAAAAAAAAAAAAAAAAAAAAAAAAAAAAAAAAAAAAAAAAAAAAAAAAAAAAAA"
+			"AAAAAAAAAAAAAAAAAAAAAAAAAAAAAAAAAAAAAAAAAAAAAAAAAAAAAAAAAAAAAAAAAAAAAAAAAAAA"
+			"AAAAAAAAAAAAAAAAAAAAAAAAAAAAAAAAAAAAAAAAAAAAAAAAAAAAAAAAAAAAAAAAAAAAAAAAAAAA"
+			"AAAAAAAAAAAAAAAAAAAAAAAAAAAAAAAAAAAAAAAAAAAAAAAAAAAAAAAAAAAAAAAAAAAAAAAAAAAA"
+			"AAAAAAAAAAAAAAAAAAAAAAAAAAAAAAAAAAAAAAAAAAAAAAAAAAAAAAAAAAAAAAAAAAAAAAAAAAAA"
+			"AAAAAAAAAAAAAAAAAAAAAAAAAAAAAAAAAAAAAAAAAAAAAAAAAAAAAAAAAAAAAAAAAAAAAAAAAAAA"
+			"AAAAAAAAAAAAAAAAAAAAAAAAAAAAAAAAAAAAAAAAAAAAAAAAAAAAAAAAAAAAAAAAAAAAAAAAAAAA"
+			"AAAAAAAAAAAAAAAAAAAAAAAAAAAAAAAAAAAAAAAAAAAAAAAAAAAAAAAAAAAAAAAAAAAAAAAAAAAA"
+			"AAAAAAAAAAAAAAAAAAAAAAAAAAAAAAAAAAAAAAAAAAAAAAAAAAAAAAAAAAAAAAAAAAAAAAAAAAAA"
+			"AAAAAAAAAAAAAAAAAAAAAAAAAAAAAAAAAAAAAAAAAAAAAAAAAAAAAAAAAAAAAAAAAAAAAAAAAAAA"
+			"AAAAAAAAAAAAAAAAAAAAAAAAAAAAAAAAAAAAAAAAAAAAAAAAAAAAAAAAAAAAAAAAAAAAAAAAAAAA"
+			"AAAAAAAAAAAAAAAAAAAAAAAAAAAAAAAAAAAAAAAAAAAAAAAAAAAAAAAAAAAAAAAAAAAAAAAAAAAA"
+			"AAAAAAAAAAAAAAAAAAAAAAAAAAAAAAAAAAAAAAAAAAAAAAAAAAAAAAAAAAAAAAAAAAAAAAAAAAAA"
+			"AAAAAAAAAAAAAAAAAAAAAAAAAAAAAAAAAAAAAAAAAAAAAAAAAAAAAAAAAAAAAAAAAAAAAAAAAAAA"
+			"AAAAAAAAAAAAAAAAAAAAAAAAAAAAAAAAAAAAAAAAAAAAAAAAAAAAAAAAAAAAAAAAAAAAAAAAAAAA"
+			"AAAAAAAAAAAAAAAAAAAAAAAAAAAAAAAAAAAAAAAAAAAAAAAAAAAAAAAAAAAAAAAAAAAAAAAAAAAA"
+			"AAAAAAAAAAAAAAAAAAAAAAAAAAAAAAAAAAAAAAAAAAAAAAAAAAAAAAAAAAAAAAAAAAAAAAAAAAAA"
+			"AAAAAAAAAAAAAAAAAAAAAAAAAAAAAAAAAAAAAAAAAAAAAAAAAAAAAAAAAAAAAAAAAAAAAAAAAAAA"
+			"AAAAAAAAAAAAAAAAAAAAAAAAAAAAAAAAAAAAAAAAAAAAAAAAAAAAAAAAAAAAAAAAAAAAAAAAAAAA"
 			"AAAAAAAAAAAAAAAAAAAAAAAAAAAAAAAAAAAAAAAAAAAAAAAAAAAAAAAAAAAAAA=="
 		)
@@
 			"UdMVAa2JxeKjR49quhYAqA3ELfCuOByOpaWlSCTasWOHpusC2sXn8+FWGGgHjCCIjnMB0L6ysrK8"
 			"vDzZi08Ygd6KQqE4OTnByHigBSBuAQAA6EtgPCEAAIC+BOIWAACAvgTiFgAAgL4E4hYAAIC+BOIW"
-			"AACAvgTiFgAAgL4E4hYAAIC+5P8BkwLNlkIXoWcAAAAASUVORK5CYII="
+			"AACAvgTiFgAAgL4E4hYAAIC+5P8BkwLNlkIXoWcAAAAASUVORK5CYIJBQUFBQUFBQUFBQUFBQUFB"
+			"QUFBQUFBQUFBQUFBQUFBQUFBQUFBQUFBQUFBQUFBQUFBQUFBQUFBQUFBQUFBQUFBQUFBQUFBQUFB"
+			"QUFBQUFBQUFBQUFBQUFBQUFBQUFBQUFBQUFBQUFBQUFBQUFBQUFBQUFBQUFBQUFBQUFBQUFBQUFB"
+			"QUFBQUFBQUFBQUFBQUFBQUFBQUFBQUFBQUFBQUFBQUFBQUFBQUFBQUFBQUFBQUFBQUFBQUFBQUFB"
+			"QUFBQUFBQUFBQUFBQUFBQUFBQUFBQUFBQUFBQUFBQUFBQUFBQUFBQUFBQUFBQUFBQUFBQUFBQUFB"
+			"QUFBQUFBQUFBQUFBQUFBQUFBQUFBQUFBQUFBQUFBQUFBQUFBQUFBQUFBQUFBQUFBQUFBQUFBQUFB"
+			"QUFBQUFBQUFBQUFBQUFBQUFBQUFBQUFBQUFBQUFBQUFBQUFBQUFBQUFBQUFBQUFBQUFBQUFBQUFB"
+			"QUFBQUFBQUFBQUFBQUFBQUFBQUFBQUFBQUFBQUFBQUFBQUFBQUFBQUFBQUFBQUFBQUFBQUFBQUFB"
+			"QUFBQUFBQUFBQUFBQUFBQUFBQUFBQUFBQUFBQUFBQUFBQUFBQUFBQUFBQUFBQUFBQUFBQUFBQUFB"
+			"QUFBQUFBQUFBQUFBQUFBQUFBQUFBQUFBQUFBQUFBQUFBQUFBQUFBQUFBQUFBQUFBQUFBQUFBQUFB"
+			"QUFBQUFBQUFBQUFBQUFBQUFBQUFBQUFBQUFBQUFBQUFBQUFBQUFBQUFBQUFBQUFBQUFBQUFBQUFB"
+			"QUFBQUFBQUFBQUFBQUFBQUFBQUFBQUFBQUFBQUFBQUFBQUFBQUFBQUFBQUFBQUFBQUFBQUFBQUFB"
+			"QUFBQUFBQUFBQUFBQUFBQUFBQUFBQUFBQUFBQUFBQUFBQUFBQUFBQUFBQUFBQUFBQUFBQUFBQUFB"
+			"QUFBQUFBQUFBQUFBQUFBQUFBQUFBQUFBQUFBQUFBQUFBQUFBQUFBQUFBQUFBQUFBQUFBQUFBQUFB"
+			"QUFBQUFBQUFBQUFBQUFBQUFBQUFBQUFBQUFBQUFBQUFBQUFBQUFBQUFBQUFBQUFBQUFBQUFBQUFB"
+			"QUFBQUFBQUFBQUFBQUFBQUFBQUFBQUFBQUFBQUFBQUFBQUFBQUFBQUFBQUFBQUFBQUFBQUFBQUFB"
+			"QUFBQUFBQUFBQUFBQUFBQUFBQUFBQUFBQUFBQUFBQUFBQUFBQUFBQUFBQUFBQUFBQUFBQUFBQUFB"
+			"QUFBQUFBQUFBQUFBQUFBQUFBQUFBQUFBQUFBQUFBQUFBQUFBQUFBQUFBQUFBQUFBQUFBQUFBQUFB"
+			"QUFBQUFBQUFBQUFBQUFBQUFBQUFBQUFBQUFBQUFBQUFBQUFBQUFBQQ=="
 		)
 	)
@@
 			"AAAAAAAAAAAAAAAAAAAAAAAAAAAAAAAAAAAAAAAAAAAAAAAAAAAAAAAAAAAAAAAAAAAAAAAAAAAA"
 			"AAAAAAAAAAAAAAAAAAAAAAAAAAAAAAAAAAAAAAAAAAAAAAAAAAAAAAAAAAAAAAAAAAAAAAAAAAAA"
-			"AAAAAAAAAAAAAAAAAAAAAAAAAAAAAAAAAAAAAAAAAAAAAAAAAAAAAAAAAA=="
+			"AAAAAAAAAAAAAAAAAAAAAAAAAAAAAAAAAAAAAAAAAAAAAAAAAAAAAAAAANYBAABAAAAAAAAAAP//"
+			"//8AAAAAAAAAAAAAAAAAAAAAAAAAAAAAAAAAAAAASL3clPh/AAAAAAAAAAAAAP////8AAAAAcNE0"
+			"CssBAAAAAAAAAAAAAAAAAAAAAAAA/////xAAAAAAAAAAAAAAAOqaw5T4fwAAAQAAAAYAAABg0jQK"
+			"ywEAAHDRNArLAQAAAAAAAAAAAAAAAAAA1wEAAEAAAAAAAAAA/////wAAAAAAAAAAAAAAAAAAAAAA"
+			"AAAAAAAAAAAAAABIvdyU+H8AAAAAAAAAAAAA/////wAAAAAI0jQKywEAAAAAAAAAAAAAAAAAAAAA"
+			"AAD/////EAAAAAAAAAAAAAAA6prDlPh/AAABAAAAAQAAAPjSNArLAQAAcNE0CssBAAAAAAAAAAAA"
+			"AAAAAADYAQAAQAAAAAAAAAD/////AAAAAAAAAAAAAAAAAAAAAAAAAAAAAAAAAAAAAEi93JT4fwAA"
+			"AAAAAAAAAAD/////AAAAAKDSNArLAQAAAAAAAAAAAAAAAAAAAAAAAP////8QAAAAAAAAAAAAAADY"
+			"ANyU+H8AAAEAAAAGAAAAsNQ0CssBAADIsTQKywEAACCyNArLAQAA//////////8AAAAAAAAAAAEA"
+			"AAAAAAAA/wAAAAAAAAD/AAAAAAAAAAAAAAAAAAAABAAAAAAAAABgCUQKywEAAAAAAAAAAAAAAAHc"
+			"lPh/AAACAAAAAAAAALDUNArLAQAAAAAAAAAAAACgA1doywEAAAAAAAAAAAAAAAAAAAAAAAAAAAAA"
+			"AAAAAP8AAAAAAAAAAAAAAAAAAAAAAAAAAAAAAAAAAAAAAAEAMCfdlPh/AAAIAAAAAQAAAAYAAAAA"
+			"AAAARwAIAiYCAAACAAAAAQAAAAAAAAAAAAAAAAAAAAAAAAAAAAAAAAAAAAAAAAAIAAAAAQAAAAAA"
+			"AAAgvdyU+H8AAAAAAAAAAAAAsNQ0CssBAAAAAAAAAAAAAAAAAAAAAAAAAAAAAAAAAAAAAAAAAAAA"
+			"AAAAAAAAAAAA/wAAAAAAAAAAAAAAAAAAAEcACAIAAAAACJTclPh/AABUAAAAAAAAAOCsNwrLAQAA"
+			"ONM0CssBAABY1DQKywEAAIB+NArLAQAAqNM0CssBAAAAAAAAAAAAAAAAAAAAAAAAAAAQAAAAAAAA"
+			"AAAAAAAAAAAAAAAAAAAAgJDsf8sBAABwkOx/ywEAAOCWNArLAQAAAAAAAAAAAACAkOx/ywEAAHCQ"
+			"7H/LAQAAAJc0CssBAAAHAAAAAAAAABYAAABNAwAAAAAAAAAAAABIJgAAAAAAAAAACAAAAAAA8DZE"
+			"CssBAACXAwAAAAAAAEDcVmjLAQAAAAAAAAAAAAAI1DQKywEAAAAAAAAAAA=="
 		)
 	)
@@
 	)
 	(symbol
+		(lib_id "power:+3.3V")
+		(at 143.51 173.99 0)
+		(mirror y)
+		(unit 1)
+		(exclude_from_sim no)
+		(in_bom yes)
+		(on_board yes)
+		(dnp no)
+		(fields_autoplaced yes)
+		(property "Reference" "#PWR07"
+			(at 143.51 177.8 0)
+			(effects
+				(font
+					(size 1.27 1.27)
+				)
+				(hide yes)
+			)
+		)
+		(property "Value" "+3.3V"
+			(at 143.51 168.91 0)
+			(effects
+				(font
+					(size 1.27 1.27)
+				)
+			)
+		)
+		(property "Footprint" ""
+			(at 143.51 173.99 0)
+			(effects
+				(font
+					(size 1.27 1.27)
+				)
+				(hide yes)
+			)
+		)
+		(property "Datasheet" ""
+			(at 143.51 173.99 0)
+			(effects
+				(font
+					(size 1.27 1.27)
+				)
+				(hide yes)
+			)
+		)
+		(property "Description" "Power symbol creates a global label with name \"+3.3V\""
+			(at 143.51 173.99 0)
+			(effects
+				(font
+					(size 1.27 1.27)
+				)
+				(hide yes)
+			)
+		)
+		(pin "1"
+		)
+		(instances
+			(project "M032FC1AE"
+				(path "/9633d16f-39f7-44d5-a160-e82bbce43a12"
+					(reference "#PWR07")
+					(unit 1)
+				)
+			)
+		)
+	)
+	(symbol
 		(lib_id "Regulator_Linear:AMS1117-3.3")
 		(at 129.54 177.8 0)
@@
 			)
 		)
-		(property "Footprint" "Package_TO_SOT_THT:TO-92_Inline"
+		(property "Footprint" "Package_TO_SOT_SMD:TSOT-23"
 			(at 92.71 125.095 0)
 			(effects

Commit message: ffffddd
Change-Id: I1eeee01593b08b9acbec1eab3a106692ce76c6c6
Parts:
- removed J7: Conn_02x08_Odd_Even, Socket:DIP_Socket-16_W4.3_W5.08_W7.62_W10.16_W10.9_3M_216-3340-00-0602J, symbol Connector_Generic:Conn_02x08_Odd_Even
- added J7: Conn_02x08_Counter_Clockwise, Socket:DIP_Socket-16_W4.3_W5.08_W7.62_W10.16_W10.9_3M_216-3340-00-0602J, symbol Connector_Generic:Conn_02x08_Counter_Clockwise
Connections:
- net isci1_clk is gone; now on net usci1_clk: J1.8 (Pin_8)
- net GND: now also J7.4 (Pin_4), J7.8 (Pin_8)
- net VCC: now also J7.12 (Pin_12), J7.16 (Pin_16)
- net spi_clk: now also J7.14 (Pin_14)
- net spi_miso: now also J7.2 (Pin_2)
- net spi_mosi: now also J7.13 (Pin_13)
- net spi_ss: now also J7.1 (Pin_1)
- net usci1_clk: now also J7.10 (Pin_10)
- net usci1_data: now also J7.9 (Pin_9)
- net at R11.1: now also J7.11 (Pin_11)
- net at R9.2: now also J7.6 (Pin_6)
- net at R10.2: now also J7.7 (Pin_7)
- net at R7.1: now also J7.15 (Pin_15)
- net at R6.2: now also J7.3 (Pin_3)
- net at R8.2: now also J7.5 (Pin_5)

Commit message: dfdfdfdf
Change-Id: I4bedd6ca326a9b17d3d6f978c0846dd558e38f70
Connections:
- net spi_miso: now also J1.5 (Pin_5), J7.13 (Pin_13); no longer J1.4 (Pin_4), J7.2 (Pin_2)
- net spi_mosi: now also J1.4 (Pin_4), J7.2 (Pin_2); no longer J1.5 (Pin_5), J7.13 (Pin_13)

Commit message: lalala
Change-Id: I877491cc6b06ae896878915a1c7d8004ea38277d
Connections:
- net spi_miso: now also J7.2 (Pin_2); no longer J7.13 (Pin_13)
- net spi_mosi: now also J7.13 (Pin_13); no longer J7.2 (Pin_2)
Other:
- moved on the sheet: D1, Q1, R1, R2, SW2
